Commit message: get the allegro visualization running

File: manipulation/models/allegro_hand_description/urdf/allegro_hand_description_left.urdf (robot description, URDF)
Before this commit: robot allegro_hand_left, 22 links, 21 joints
Links:
- link link_0: geometry collision box size=0.0196 0.0275 0.0164; visual mesh filename=../meshes/link_0.0.obj
- link link_1: geometry collision box size=0.0196 0.0275 0.054; visual mesh filename=../meshes/link_1.0.obj
- link link_10: geometry collision box size=0.0196 0.0275 0.0384; visual mesh filename=../meshes/link_2.0.obj
- link link_11: geometry collision box size=0.0196 0.0275 0.0267; visual mesh filename=../meshes/link_3.0.obj
- link link_11_tip: geometry collision sphere radius=0.012; visual mesh filename=../meshes/link_3.0_tip.obj
- link link_12: geometry collision box size=0.0358 0.034 0.0455; visual mesh filename=../meshes/link_12.0_left.obj
- link link_13: geometry collision box size=0.0196 0.0275 0.0177; visual mesh filename=../meshes/link_13.0.obj
- link link_14: geometry collision box size=0.0196 0.0275 0.0514; visual mesh filename=../meshes/link_14.0.obj
- link link_15: geometry collision box size=0.0196 0.0275 0.0423; visual mesh filename=../meshes/link_15.0.obj
- link link_15_tip: geometry collision sphere radius=0.012; visual mesh filename=../meshes/link_15.0_tip.obj
- link link_2: geometry collision box size=0.0196 0.0275 0.0384; visual mesh filename=../meshes/link_2.0.obj
- link link_3: geometry collision box size=0.0196 0.0275 0.0267; visual mesh filename=../meshes/link_3.0.obj
- link link_3_tip: geometry collision sphere radius=0.012; visual mesh filename=../meshes/link_3.0_tip.obj
- link link_4: geometry collision box size=0.0196 0.0275 0.0164; visual mesh filename=../meshes/link_0.0.obj
- link link_5: geometry collision box size=0.0196 0.0275 0.054; visual mesh filename=../meshes/link_1.0.obj
- link link_6: geometry collision box size=0.0196 0.0275 0.0384; visual mesh filename=../meshes/link_2.0.obj
- link link_7: geometry collision box size=0.0196 0.0275 0.0267; visual mesh filename=../meshes/link_3.0.obj
- link link_7_tip: geometry collision sphere radius=0.012; visual mesh filename=../meshes/link_3.0_tip.obj
- link link_8: geometry collision box size=0.0196 0.0275 0.0164; visual mesh filename=../meshes/link_0.0.obj
- link link_9: geometry collision box size=0.0196 0.0275 0.054; visual mesh filename=../meshes/link_1.0.obj
- link palm_link: geometry collision box size=0.0408 0.1130 0.095; visual mesh filename=../meshes/base_link_left.obj

Commit message: added actuators to the allegro hand's urdf files

File: manipulation/models/allegro_hand_description/urdf/allegro_hand_description_left.urdf (robot description, URDF)
Before this commit: robot allegro_hand_left, 22 links, 21 joints
Joints:
- joint joint_0: origin xyz=0 -0.0435 -0.001542 rpy=0.08726646255 0 0 -> xyz=0 0.0435 -0.001542 rpy=-0.08726646255 0 0
- joint joint_12: axis +1 0 0 -> 1 0 0
- joint joint_8: origin xyz=0 0.0435 -0.001542 rpy=-0.08726646255 0 0 -> xyz=0 -0.0435 -0.001542 rpy=0.08726646255 0 0

File: manipulation/models/allegro_hand_description/urdf/allegro_hand_description_left_backup.urdf (robot description, URDF)
Before this commit: robot allegro_hand_right, 22 links, 21 joints
Links:
- link link_12: geometry collision box size=0.0358 0.034 0.0455; visual mesh filename=../meshes/link_12.0_left.obj
- link palm_link: geometry collision box size=0.0408 0.1130 0.095; visual mesh filename=../meshes/base_link_left.obj
Joints:
- joint joint_0: origin xyz=0 0.0435 -0.001542 rpy=-0.08726646255 0 0 -> xyz=0 -0.0435 -0.001542 rpy=0.08726646255 0 0
- joint joint_12: axis -1 0 0 -> +1 0 0; origin xyz=-0.0182 0.019333 -0.045987 rpy=0 -1.65806278845 -1.5707963259 -> xyz=-0.0182 -0.019333 -0.045987 rpy=0 -1.65806278845 1.5707963259
- joint joint_13: axis 0 0 1 -> 0 0 -1; origin xyz=-0.027 0.005 0.0399 -> xyz=-0.027 -0.005 0.0399
- joint joint_8: origin xyz=0 -0.0435 -0.001542 rpy=0.08726646255 0 0 -> xyz=0 0.0435 -0.001542 rpy=-0.08726646255 0 0

Commit message: fixed all the allegro hand model files, and fixed the constant load demo file.

File: manipulation/models/allegro_hand_description/urdf/allegro_hand_description_left.urdf (robot description, URDF)
Before this commit: robot allegro_hand_left, 22 links, 21 joints
Joints:
- joint joint_0: origin xyz=0 0.0435 -0.001542 rpy=-0.08726646255 0 0 -> xyz=0 -0.0435 -0.001542 rpy=0.08726646255 0 0
- joint joint_8: origin xyz=0 -0.0435 -0.001542 rpy=0.08726646255 0 0 -> xyz=0 0.0435 -0.001542 rpy=-0.08726646255 0 0

Commit message: fix the opposite rotation axis of the left hand joints

File: manipulation/models/allegro_hand_description/urdf/allegro_hand_description_left.urdf (robot description, URDF)
Before this commit: robot allegro_hand_left, 22 links, 21 joints
Joints:
- joint joint_0: axis 0 0 1 -> 0 0 -1
- joint joint_4: axis 0 0 1 -> 0 0 -1
- joint joint_8: axis 0 0 1 -> 0 0 -1; origin xyz=0 0.0435 -0.001542 rpy=-0.08726646255 0 0 -> xyz=0 0.0435 -0.001542 rpy=0.08726646255 0 0

Commit message: updated the model files with the public version

File: manipulation/models/allegro_hand_description/urdf/allegro_hand_description_left.urdf (robot description, URDF)
Before this commit: robot allegro_hand_left, 22 links, 21 joints
Joints:
- joint joint_0: limit lower=-0.47 upper=0.47 effort=15 velocity=7 -> lower=-0.47 upper=0.47 effort=0.7 velocity=7
- joint joint_1: limit lower=-0.196 upper=1.61 effort=15 velocity=7 -> lower=-0.196 upper=1.61 effort=0.7 velocity=7
- joint joint_10: limit lower=-0.174 upper=1.709 effort=15 velocity=7 -> lower=-0.174 upper=1.709 effort=0.7 velocity=7
- joint joint_11: limit lower=-0.227 upper=1.618 effort=15 velocity=7 -> lower=-0.227 upper=1.618 effort=0.7 velocity=7
- joint joint_12: limit lower=0.263 upper=1.396 effort=15 velocity=7 -> lower=0.263 upper=1.396 effort=0.7 velocity=7
- joint joint_13: limit lower=-0.105 upper=1.163 effort=15 velocity=7 -> lower=-0.105 upper=1.163 effort=0.7 velocity=7
- joint joint_14: limit lower=-0.189 upper=1.644 effort=15 velocity=7 -> lower=-0.189 upper=1.644 effort=0.7 velocity=7
- joint joint_15: limit lower=-0.162 upper=1.719 effort=15 velocity=7 -> lower=-0.162 upper=1.719 effort=0.7 velocity=7
- joint joint_2: limit lower=-0.174 upper=1.709 effort=15 velocity=7 -> lower=-0.174 upper=1.709 effort=0.7 velocity=7
- joint joint_3: limit lower=-0.227 upper=1.618 effort=15 velocity=7 -> lower=-0.227 upper=1.618 effort=0.7 velocity=7
- joint joint_4: limit lower=-0.47 upper=0.47 effort=15 velocity=7 -> lower=-0.47 upper=0.47 effort=0.7 velocity=7
- joint joint_5: limit lower=-0.196 upper=1.61 effort=15 velocity=7 -> lower=-0.196 upper=1.61 effort=0.7 velocity=7
- joint joint_6: limit lower=-0.174 upper=1.709 effort=15 velocity=7 -> lower=-0.174 upper=1.709 effort=0.7 velocity=7
- joint joint_7: limit lower=-0.227 upper=1.618 effort=15 velocity=7 -> lower=-0.227 upper=1.618 effort=0.7 velocity=7
- joint joint_8: limit lower=-0.47 upper=0.47 effort=15 velocity=7 -> lower=-0.47 upper=0.47 effort=0.7 velocity=7
- joint joint_9: limit lower=-0.196 upper=1.61 effort=15 velocity=7 -> lower=-0.196 upper=1.61 effort=0.7 velocity=7

File: manipulation/models/allegro_hand_description/urdf/allegro_hand_description_right.urdf (robot description, URDF)
Before this commit: robot allegro_hand_right, 22 links, 21 joints
Joints:
- joint joint_0: limit lower=-0.47 upper=0.47 effort=15 velocity=7 -> lower=-0.47 upper=0.47 effort=0.7 velocity=7
- joint joint_1: limit lower=-0.196 upper=1.61 effort=15 velocity=7 -> lower=-0.196 upper=1.61 effort=0.7 velocity=7
- joint joint_10: limit lower=-0.174 upper=1.709 effort=15 velocity=7 -> lower=-0.174 upper=1.709 effort=0.7 velocity=7
- joint joint_11: limit lower=-0.227 upper=1.618 effort=15 velocity=7 -> lower=-0.227 upper=1.618 effort=0.7 velocity=7
- joint joint_12: limit lower=0.263 upper=1.396 effort=15 velocity=7 -> lower=0.263 upper=1.396 effort=0.7 velocity=7
- joint joint_13: limit lower=-0.105 upper=1.163 effort=15 velocity=7 -> lower=-0.105 upper=1.163 effort=0.7 velocity=7
- joint joint_14: limit lower=-0.189 upper=1.644 effort=15 velocity=7 -> lower=-0.189 upper=1.644 effort=0.7 velocity=7
- joint joint_15: limit lower=-0.162 upper=1.719 effort=15 velocity=7 -> lower=-0.162 upper=1.719 effort=0.7 velocity=7
- joint joint_2: limit lower=-0.174 upper=1.709 effort=15 velocity=7 -> lower=-0.174 upper=1.709 effort=0.7 velocity=7
- joint joint_3: limit lower=-0.227 upper=1.618 effort=15 velocity=7 -> lower=-0.227 upper=1.618 effort=0.7 velocity=7
- joint joint_4: limit lower=-0.47 upper=0.47 effort=15 velocity=7 -> lower=-0.47 upper=0.47 effort=0.7 velocity=7
- joint joint_5: limit lower=-0.196 upper=1.61 effort=15 velocity=7 -> lower=-0.196 upper=1.61 effort=0.7 velocity=7
- joint joint_6: limit lower=-0.174 upper=1.709 effort=15 velocity=7 -> lower=-0.174 upper=1.709 effort=0.7 velocity=7
- joint joint_7: limit lower=-0.227 upper=1.618 effort=15 velocity=7 -> lower=-0.227 upper=1.618 effort=0.7 velocity=7
- joint joint_8: limit lower=-0.47 upper=0.47 effort=15 velocity=7 -> lower=-0.47 upper=0.47 effort=0.7 velocity=7
- joint joint_9: limit lower=-0.196 upper=1.61 effort=15 velocity=7 -> lower=-0.196 upper=1.61 effort=0.7 velocity=7
